Commit message: Updated fr3_gazebo.urdf.xacro - fr3_finger_joint2

File: src/franka_sim/urdf/fr3_gazebo.urdf.xacro (robot description, xacro)
@@ -26,6 +26,13 @@
     <xacro:fr3_arm_joint name="fr3_joint6" initial="${pi/2}"/>
     <xacro:fr3_arm_joint name="fr3_joint7" initial="${pi/4}"/>
-    <!-- Chwytak: tylko joint1, joint2 mimic -->
+    <!-- Chwytak: jawne sterowanie oboma palcami (Opcja A — mimic niewspierany w DART) -->
     <joint name="fr3_finger_joint1">
+      <command_interface name="position"/>
+      <state_interface name="position">
+        <param name="initial_value">0.0</param>
+      </state_interface>
+      <state_interface name="velocity"/>
+    </joint>
+    <joint name="fr3_finger_joint2">
       <command_interface name="position"/>
       <state_interface name="position">

Commit message: Robot attached to the ground - URDF

File: src/franka_sim/urdf/fr3_gazebo.urdf.xacro (robot description, xacro)
@@ -3,4 +3,11 @@
   <!-- 1. Bazowy opis — BEZ ros2_control:=true -->
   <xacro:include filename="$(find franka_description)/robots/fr3/fr3.urdf.xacro"/>
+  <!-- 1a. Przyczepienie robota do podłoża -->
+  <link name="world"/>
+  <joint name="world_to_base" type="fixed">
+    <parent link="world"/>
+    <child link="base"/>
+    <origin xyz="0 0 0" rpy="0 0 0"/>
+  </joint>
   <!-- 2. Makro na jeden staw ramienia -->
   <xacro:macro name="fr3_arm_joint" params="name initial">
